File: Eagle/ProjV1.brd (EAGLE design)
At the start: 94.9 x 63.5 mm, 24 parts, among them IC1 CD4007UBM, IC2 CD4007UBM, IC3 CD4007UBM, SW1 EC12E_SW, U1 MIC5504-3.3YM5-T5, U2 MCP2200-I/SS, U3 ATMEGA328PB-AU, Y1 16MHz

Commit message: Schematic Changes
Added votage and ground flags and switched to running board at 3.3V
Parts:
- Y1: value 16MHz -> 12MHz
Connections:
- removed net 3.3V: C2.1, T3.1, U1.5
- removed net GND: IC1.4, IC1.7, IC2.4, IC2.7, IC2.9, IC3.4, IC3.7, IC3.9
- removed net N$31: U3.18
- removed net VBUS: C3.1, CN1.VBUS, T1.1, T2.1, U$1.2, U1.1, U1.3, U2.1
- new net +5V: C3.1, CN1.VBUS, T1.1, T2.1, U1.1, U1.3, U2.1
- net 0: now also IC1.4, IC1.7, IC2.4, IC2.7, IC2.9, IC3.4, IC3.7, IC3.9
- net VCC: now also C2.1, T3.1, U$1.2, U1.5, U3.18
Routing:
- net VBUS: track 58.5 -> 0.00 mm
- net +5V: track 0.00 -> 50.4 mm
- net 3.3V: track 11.3 -> 0.00 mm
- net VCC: track 36.6 -> 46.7 mm
