File: ProjV3.sch (EAGLE design)
At the start: 30 parts, among them IC1 CD4007UBM, IC2 CD4007UBM, IC3 CD4007UBM, U1 MIC5504-3.3YM5-T5, U2 MCP2200-I/MQ, U3 ATMEGA328PB-AU, U4 EN11-HSM1BF20, Y1 CSTNE12M0G55A000R0

Commit message: Added copies of old versions
Updated version numbers and add old versions for comparison and report writing
Parts:
- removed R1, R2, R3, R4: 10k, rcl:R-US_R0805
- removed T5, T6: (no value), zetex:NMOSSOT23
- U2: value MCP2200-I/MQ -> MCP2200-I/SS; device MCP2200-I_MQ:MCP2200-I/MQ -> MCP2200-I_SS:MCP2200-I/SS
- Y1: value CSTNE12M0G55A000R0 -> 12MHz; device CSTNE12M0G55A000R0:CSTNE12M0G55A000R0 -> SparkFun-Clocks:RESONATOR-16MHZSMD_3.2X1.3
Connections:
- net N$10 renamed RX/TX
- net N$11 renamed TX/RX
- removed net +3V3: C2.1, R2.2, R4.2, T3.D, T5.G, T6.G, U$1.VCC, U1.VOUT
- removed net N$16: R2.1, T5.S, U$1.SDA
- removed net N$19: R4.1, T6.S, U$1.SCL
- removed net N$7: C1.1, U2.VUSB
- new net VCC: C1.1, C2.1, ISP1.VCC, T3.D, U$1.VCC, U1.VOUT, U2.VDD, U2.VUSB, U3.AVCC, U3.VCC
- net +5V: no longer ISP1.VCC, R1.2, R3.2, U2.VDD, U3.AVCC, U3.VCC
- net 0: now also Y1.2; no longer U2.!RST, U2.EXP, U2.VSS, Y1.GND
- net C4: now also IC2.Q1_(N)_DRAIN, IC2.Q1_(P)_SOURCE; no longer IC2.Q2_(N)_DRAIN, IC2.Q2_(P)_DRAIN
- net C5: now also IC2.Q2_(N)_DRAIN, IC2.Q2_(P)_DRAIN; no longer IC2.Q1_(N)_DRAIN, IC2.Q1_(P)_SOURCE
- net D+: now also U2.D+; no longer U2.GP6/RXLED
- net D-: now also U2.D-; no longer U2.GP7/TXLED
- net LC4: now also IC2.Q1_GATES; no longer IC2.Q2_GATES
- net LC5: now also IC2.Q2_GATES; no longer IC2.Q1_GATES
- net N$14: now also Y1.3; no longer Y1.INPUT
- net N$6: now also Y1.1; no longer Y1.OUTPUT
- net SCL: now also U$1.SCL; no longer R3.1, T6.D
- net SDA: now also U$1.SDA; no longer R1.1, T5.D
Other:
- moved on the sheet: C1
