File: ProjV5.brd (EAGLE design)
At the start: 63.4 x 46.9 mm, 33 parts, among them IC1 CD4007UBM, IC2 CD4007UBM, IC3 CD4007UBM, U1 MIC5504-3.3YM5-T5, U2 MCP2200-I/MQ, U3 ATMEGA328PB-AU, U4 EN11-HSM1BF20, Y1 CSTNE12M0G55A000R0

Commit message: Added copies of old versions
Updated version numbers and add old versions for comparison and report writing
Parts:
- moved Y1 0.06 mm to (33.3, 42.3)
Routing:
- net 0: track 0.00 -> 23.3 mm, vias 0 -> 24
- net LEDA: track 61.3 -> 58.9 mm
- net C1: track 22.3 -> 23.8 mm
- net LED5: track 33.4 -> 32.8 mm
- added copper zone on layer 16, net 0
- removed copper zone on layer 16, net 1
