File: ProjV5.brd (EAGLE design)
At the start: 62.9 x 50.1 mm, 33 parts, among them IC1 CD4007UBM, IC2 CD4007UBM, IC3 CD4007UBM, U1 MIC5504-3.3YM5-T5, U2 MCP2200-I/MQ, U3 ATMEGA328PB-AU, U4 EN11-HSM1BF20, Y1 CSTNE12M0G55A000R0

Commit message: Update In Case of Missed Changes
Parts:
- moved USB1 1.15 mm to (58.7, 32.8)
Routing:
- net 0: track 26.3 -> 24.0 mm
- net D+: track 36.3 -> 37.5 mm
- net D-: track 32.1 -> 33.3 mm
- net +5V: track 183.8 -> 184.9 mm
Other:
- board size 62.9 x 50.1 mm -> 62.4 x 50.3 mm
Changed lines of the file:
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@@
 <layer number="25" name="tNames" color="7" fill="1" visible="yes" active="yes"/>
 <layer number="26" name="bNames" color="7" fill="1" visible="yes" active="yes"/>
-<layer number="27" name="tValues" color="7" fill="1" visible="no" active="yes"/>
+<layer number="27" name="tValues" color="7" fill="1" visible="yes" active="yes"/>
 <layer number="28" name="bValues" color="7" fill="1" visible="no" active="yes"/>
 <layer number="29" name="tStop" color="7" fill="3" visible="no" active="yes"/>
@@
 <board>
 <plain>
-<wire x1="1.15" y1="-2.33" x2="63.95" y2="-2.36" width="0" layer="20"/>
-<wire x1="63.95" y1="-2.36" x2="63.88" y2="47.675" width="0" layer="20"/>
-<wire x1="63.88" y1="47.675" x2="1.08" y2="47.705" width="0" layer="20"/>
+<wire x1="1.15" y1="-2.33" x2="63.5" y2="-2.56" width="0" layer="20"/>
+<wire x1="63.5" y1="-2.56" x2="63.43" y2="47.475" width="0" layer="20"/>
+<wire x1="63.43" y1="47.475" x2="1.08" y2="47.705" width="0" layer="20"/>
 <wire x1="1.08" y1="47.705" x2="1.15" y2="-2.33" width="0" layer="20"/>
 <text x="58.02" y="9.66" size="1.778" layer="22" rot="MR0">Marcel Vieira 11/12/20 Version 4</text>
@@
 <attribute name="NAME" x="28.755" y="42.25" size="1.27" layer="25" rot="R180" align="center"/>
 </element>
-<element name="USB1" library="usbFromLCSC" package="C77238" value="C77238" x="57.51" y="32.91" smashed="yes">
-<attribute name="NAME" x="57.764" y="41.8" size="1.016" layer="25"/>
+<element name="USB1" library="usbFromLCSC" package="C77238" value="C77238" x="58.66" y="32.835" smashed="yes">
+<attribute name="NAME" x="58.914" y="41.725" size="1.016" layer="25"/>
 </element>
 <element name="U$2" library="dicons" package="FIDUCIAL_G15S" value="" x="2.8325" y="-0.27415" smashed="yes"/>
@@
 <wire x1="41.10813125" y1="36.4478" x2="40.7378" y2="36.81813125" width="0.2032" layer="16"/>
 <contactref element="USB1" pad="3"/>
-<wire x1="57.754475" y1="36.9780625" x2="54.84600625" y2="36.9780625" width="0.2032" layer="1"/>
-<wire x1="54.84600625" y1="36.9780625" x2="54.53186875" y2="37.2922" width="0.2032" layer="1"/>
+<wire x1="58.904475" y1="36.9030625" x2="54.92100625" y2="36.9030625" width="0.2032" layer="1"/>
+<wire x1="54.92100625" y1="36.9030625" x2="54.53186875" y2="37.2922" width="0.2032" layer="1"/>
 <wire x1="53.24186875" y1="37.2922" x2="52.78526875" y2="37.7488" width="0.2032" layer="1"/>
 <wire x1="54.53186875" y1="37.2922" x2="53.24186875" y2="37.2922" width="0.2032" layer="1"/>
@@
 <contactref element="USB1" pad="2"/>
 <wire x1="54.27" y1="36.66" x2="54.63" y2="36.3" width="0.2032" layer="1"/>
-<wire x1="57.72665" y1="36.3" x2="57.754475" y2="36.327825" width="0.2032" layer="1"/>
-<wire x1="54.63" y1="36.3" x2="57.72665" y2="36.3" width="0.2032" layer="1"/>
+<wire x1="58.8573" y1="36.3" x2="58.904475" y2="36.252825" width="0.2032" layer="1"/>
+<wire x1="54.63" y1="36.3" x2="58.8573" y2="36.3" width="0.2032" layer="1"/>
 <wire x1="52.89" y1="36.63" x2="54.24" y2="36.63" width="0.2032" layer="16"/>
 </signal>
@@
 <wire x1="40.59" y1="13.44" x2="40.59" y2="7.83" width="0.4064" layer="1"/>
 <wire x1="35.51" y1="18.52" x2="35.51" y2="20.74" width="0.4064" layer="1"/>
-<wire x1="35.51" y1="18.52" x2="38.2525" y2="15.7775" width="0.4064" layer="1"/>
-<wire x1="38.2525" y1="15.7775" x2="40.59" y2="13.44" width="0.4064" layer="1"/>
+<wire x1="35.51" y1="18.52" x2="40.59" y2="13.44" width="0.4064" layer="1"/>
 <wire x1="53.78564375" y1="36.03" x2="52.41" y2="36.03" width="0.4064" layer="1"/>
 <wire x1="54" y1="33.3" x2="54" y2="35.58" width="0.4064" layer="1"/>
@@
 <wire x1="54" y1="35.81564375" x2="53.78564375" y2="36.03" width="0.4064" layer="1"/>
 <contactref element="USB1" pad="1"/>
-<wire x1="57.754475" y1="35.677584375" x2="54.097584375" y2="35.677584375" width="0.4064" layer="1"/>
-<wire x1="54.097584375" y1="35.677584375" x2="54" y2="35.58" width="0.4064" layer="1"/>
+<wire x1="58.904475" y1="35.602584375" x2="54.022584375" y2="35.602584375" width="0.4064" layer="1"/>
+<wire x1="54.022584375" y1="35.602584375" x2="54" y2="35.58" width="0.4064" layer="1"/>
 <wire x1="57.78" y1="29.65723125" x2="54.13723125" y2="33.3" width="0.4064" layer="1"/>
 <wire x1="54.13723125" y1="33.3" x2="54" y2="33.3" width="0.4064" layer="1"/>
@@
 <wire x1="54.58" y1="30.63" x2="54.6" y2="30.65" width="0.4064" layer="1"/>
 <via x="54.6" y="30.65" extent="1-16" drill="0.35"/>
-<wire x1="54.6" y1="30.65" x2="54.6" y2="31.375" width="0.4064" layer="16"/>
 <via x="56.6" y="40.225" extent="1-16" drill="0.35"/>
 <via x="42.675" y="40" extent="1-16" drill="0.35"/>
@@
 <wire x1="38" y1="19.125" x2="37.85" y2="19.275" width="0.4064" layer="1"/>
 <via x="38" y="18.925" extent="1-16" drill="0.35"/>
-<wire x1="38.4" y1="18.875" x2="38.05" y2="18.875" width="0.4064" layer="16"/>
-<wire x1="38" y1="18.925" x2="38.05" y2="18.875" width="0.4064" layer="16"/>
 <wire x1="49.99" y1="38.295" x2="49.975" y2="38.31" width="0.4064" layer="1"/>
 <wire x1="49.975" y1="38.31" x2="49.975" y2="39.15" width="0.4064" layer="1"/>
@@
 </polygon>
 <wire x1="53.592" y1="30.63" x2="52.205" y2="30.63" width="0.4064" layer="1"/>
-<wire x1="52.205" y1="30.63" x2="52.175" y2="30.6" width="0.4064" layer="1"/>
 <wire x1="33.325" y1="42.28" x2="33.325" y2="43.525" width="0.4064" layer="1"/>
 <via x="33.325" y="43.525" extent="1-16" drill="0.35"/>
 <via x="50.975" y="9.6" extent="1-16" drill="0.35"/>
-<wire x1="58.3346125" y1="40.22393125" x2="59.8596125" y2="38.69893125" width="0.4064" layer="1"/>
-<wire x1="59.8596125" y1="38.69893125" x2="59.8596125" y2="38.27854375" width="0.4064" layer="1"/>
-<wire x1="59.8596125" y1="38.27854375" x2="57.754475" y2="38.27854375" width="0.4064" layer="1"/>
+<wire x1="59.4846125" y1="40.14893125" x2="59.8596125" y2="39.77393125" width="0.4064" layer="1"/>
+<wire x1="59.8596125" y1="38.27854375" x2="59.8596125" y2="39.77393125" width="0.4064" layer="1"/>
 <wire x1="32.135" y1="37.965" x2="31.055" y2="37.965" width="0.4064" layer="1"/>
 <wire x1="31.055" y1="37.965" x2="31.03" y2="37.99" width="0.4064" layer="1"/>
@@
 <via x="35.15" y="24.025" extent="1-16" drill="0.35"/>
 <via x="38.725" y="23.175" extent="1-16" drill="0.35"/>
-<wire x1="37.11" y1="29.1" x2="37.11" y2="27.585" width="0.4064" layer="1"/>
 <via x="56.525" y="32.925" extent="1-16" drill="0.35"/>
 <via x="29.65" y="41.375" extent="1-16" drill="0.35"/>
@@
 <wire x1="29.65" y1="41.375" x2="29.65" y2="39.825" width="0.2032" layer="1"/>
 <wire x1="29.65" y1="39.825" x2="29.9" y2="39.575" width="0.2032" layer="1"/>
+<wire x1="58.904475" y1="38.20354375" x2="58.94831875" y2="38.1597" width="0.4064" layer="1"/>
+<wire x1="59.74076875" y1="38.1597" x2="59.8596125" y2="38.27854375" width="0.4064" layer="1"/>
+<wire x1="58.94831875" y1="38.1597" x2="59.74076875" y2="38.1597" width="0.4064" layer="1"/>
+<wire x1="38" y1="18.925" x2="38.05" y2="18.875" width="0.4064" layer="16"/>
+<wire x1="37.11" y1="29.1" x2="37.11" y2="27.215" width="0.4064" layer="1"/>
+<wire x1="37.11" y1="27.215" x2="37.175" y2="27.15" width="0.4064" layer="1"/>
 </signal>
 <signal name="N$15">
