File: ProjV5Submission.brd (EAGLE design)
At the start: 62.9 x 50.1 mm, 33 parts, among them IC1 CD4007UBM, IC2 CD4007UBM, IC3 CD4007UBM, U1 MIC5504-3.3YM5-T5, U2 MCP2200-I/MQ, U3 ATMEGA328PB-AU, U4 EN11-HSM1BF20, Y1 CSTNE12M0G55A000R0

Commit message: Renamed Files
Renamed some files ran more checks and fixed format up some more
Parts:
- moved USB1 1.15 mm to (58.7, 32.8)
Routing:
- net 0: track 26.3 -> 23.0 mm
- net +5V: track 183.8 -> 185.0 mm
- net D+: track 36.3 -> 37.5 mm
- net D-: track 32.1 -> 33.3 mm
Other:
- board size 62.9 x 50.1 mm -> 62.4 x 50.3 mm
